Commit message: updated assets

File: src/curobo/content/assets/robot/motoman/motoman.urdf (robot description, URDF)
Before this commit: robot motoman_sda10f, 36 links, 35 joints
Links:
- link camera_arm_link: geometry collision box size=0.12 0.045 0.04; visual box size=0.12 0.045 0.04
Joints:
- joint camera_arm_joint: origin xyz=0 0.06 0.1 rpy=0 0 0 -> xyz=0 -0.061 0.04 rpy=0 0 0; parent arm_right_link_6_b -> arm_right_link_7_t

File: src/curobo/content/assets/robot/motoman/sda10f.xacro (robot description, xacro)
@@ -70,5 +70,5 @@
 			<origin rpy="0 0 0" xyz="0 0 0" />
 			<geometry>
-				<box size="0.12 0.06 0.05" />
+				<box size="0.12 0.045 0.04" />
 			</geometry>
 			<material name="">
@@ -79,12 +79,12 @@
 			<origin rpy="0 0 0" xyz="0 0 0" />
 			<geometry>
-				<box size="0.12 0.06 0.05" />
+				<box size="0.12 0.045 0.04" />
 			</geometry>
 		</collision>
 	</link>
 	<joint name="camera_arm_joint" type="fixed">
-		<parent link="arm_right_link_6_b" />
+		<parent link="arm_right_link_7_t" />
 		<child link="camera_arm_link" />
-		<origin rpy="0 0 0" xyz="0 0.06 0.1" />
+		<origin rpy="0 0 0" xyz="0 -0.061 0.04" />
 	</joint>
 </robot>
